File: fimur-electrical/fimur-electrical-v0-2/fimur-electrical-v0-2.kicad_sch (KiCad schematic)
At the start: 20 parts, among them J1 Conn_01x16, J10 Conn_01x04, J11 Conn_01x04, J12 Conn_01x04, J13 Conn_01x04, J14 Conn_01x04, J15 Conn_01x04, J17 Conn_02x02_Odd_Even, J2 Conn_01x16, J3 Conn_01x03_Pin, J4 Conn_01x03_Pin, J5 Conn_01x03_Pin, J6 Conn_01x04, J7 Conn_01x04, J8 Conn_01x04, J9 Conn_01x04, U1 TCA9548APWR

Commit message: multiplex schematic and layout and standardization with 2-imu board
Parts:
- J10: renamed from J9; footprint Connector_JST:JST_PH_S4B-PH-K_1x04_P2.00mm_Horizontal -> Connector_JST:JST_SH_SM04B-SRSS-TB_1x04-1MP_P1.00mm_Horizontal
- J11: renamed from J10; footprint Connector_JST:JST_PH_S4B-PH-K_1x04_P2.00mm_Horizontal -> Connector_JST:JST_SH_SM04B-SRSS-TB_1x04-1MP_P1.00mm_Horizontal
- J12: renamed from J11; footprint Connector_JST:JST_PH_S4B-PH-K_1x04_P2.00mm_Horizontal -> Connector_JST:JST_SH_SM04B-SRSS-TB_1x04-1MP_P1.00mm_Horizontal
- J13: renamed from J12; footprint Connector_JST:JST_PH_S4B-PH-K_1x04_P2.00mm_Horizontal -> Connector_JST:JST_SH_SM04B-SRSS-TB_1x04-1MP_P1.00mm_Horizontal
- J14: renamed from J13; footprint Connector_JST:JST_PH_S4B-PH-K_1x04_P2.00mm_Horizontal -> Connector_JST:JST_SH_SM04B-SRSS-TB_1x04-1MP_P1.00mm_Horizontal
- J15: renamed from J14; footprint Connector_JST:JST_PH_S4B-PH-K_1x04_P2.00mm_Horizontal -> Connector_JST:JST_SH_SM04B-SRSS-TB_1x04-1MP_P1.00mm_Horizontal
- J17: footprint Connector_PinSocket_1.27mm:PinSocket_2x02_P1.27mm_Vertical -> Connector_PinSocket_2.54mm:PinSocket_2x02_P2.54mm_Vertical
- J6: footprint Connector_JST:JST_PH_S4B-PH-K_1x04_P2.00mm_Horizontal -> Connector_JST:JST_SH_SM04B-SRSS-TB_1x04-1MP_P1.00mm_Horizontal
- J7: renamed from J15; footprint Connector_JST:JST_PH_S4B-PH-K_1x04_P2.00mm_Horizontal -> Connector_JST:JST_SH_SM04B-SRSS-TB_1x04-1MP_P1.00mm_Horizontal
- J8: renamed from J7; footprint Connector_JST:JST_PH_S4B-PH-K_1x04_P2.00mm_Horizontal -> Connector_JST:JST_SH_SM04B-SRSS-TB_1x04-1MP_P1.00mm_Horizontal
- J9: renamed from J8; footprint Connector_JST:JST_PH_S4B-PH-K_1x04_P2.00mm_Horizontal -> Connector_JST:JST_SH_SM04B-SRSS-TB_1x04-1MP_P1.00mm_Horizontal
Connections:
- net VCC: now reaches J1.1 (3V3), J10.2 (Pin_2), J11.2 (Pin_2), J12.2 (Pin_2), J13.2 (Pin_2), J14.2 (Pin_2), J15.2 (Pin_2), J3.1 (Pin_1), J4.1 (Pin_1), J5.1 (Pin_1), J6.2 (Pin_2), J7.2 (Pin_2), J8.2 (Pin_2), J9.2 (Pin_2), R1.1, R2.1, R3.1, U1.24 (VCC)
Changed lines of the file:
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@@
 	)
 	(junction
-		(at 64.77 160.02)
+		(at 36.83 85.09)
 		(diameter 0)
 		(color 0 0 0 0)
 	)
 	(junction
-		(at 36.83 160.02)
+		(at 35.56 87.63)
+		(diameter 0)
+		(color 0 0 0 0)
+	)
+	(junction
+		(at 64.77 160.02)
 		(diameter 0)
 		(color 0 0 0 0)
@@
 	(wire
 		(pts
-			(xy 33.02 87.63) (xy 39.37 87.63)
+			(xy 33.02 87.63) (xy 35.56 87.63)
 		)
 		(stroke
@@
 	(wire
 		(pts
+			(xy 35.56 87.63) (xy 39.37 87.63)
+		)
+		(stroke
+			(width 0)
+			(type default)
+		)
+	)
+	(wire
+		(pts
 			(xy 167.64 149.86) (xy 175.26 149.86)
 		)
@@
 		(dnp no)
 		(fields_autoplaced yes)
-		(property "Reference" "J13"
+		(property "Reference" "J14"
 			(at 209.55 149.8599 0)
 			(effects
@@
 			)
 		)
-		(property "Footprint" "Connector_JST:JST_PH_S4B-PH-K_1x04_P2.00mm_Horizontal"
+		(property "Footprint" "Connector_JST:JST_SH_SM04B-SRSS-TB_1x04-1MP_P1.00mm_Horizontal"
 			(at 207.01 149.86 0)
 			(effects
@@
 			(project "fimur-electrical-v0-2"
 				(path "/d9ca54f7-b1e2-4ace-986c-e50c0b614954"
-					(reference "J13")
+					(reference "J14")
 					(unit 1)
 				)
@@
 		(dnp no)
 		(fields_autoplaced yes)
-		(property "Reference" "J14"
+		(property "Reference" "J15"
 			(at 236.22 154.9399 0)
 			(effects
@@
 			)
 		)
-		(property "Footprint" "Connector_JST:JST_PH_S4B-PH-K_1x04_P2.00mm_Horizontal"
+		(property "Footprint" "Connector_JST:JST_SH_SM04B-SRSS-TB_1x04-1MP_P1.00mm_Horizontal"
 			(at 233.68 154.94 0)
 			(effects
@@
 			(project "fimur-electrical-v0-2"
 				(path "/d9ca54f7-b1e2-4ace-986c-e50c0b614954"
-					(reference "J14")
+					(reference "J15")
 					(unit 1)
 				)
@@
 		(dnp no)
 		(fields_autoplaced yes)
-		(property "Reference" "J8"
+		(property "Reference" "J9"
 			(at 156.21 118.1099 0)
 			(effects
@@
 			)
 		)
-		(property "Footprint" "Connector_JST:JST_PH_S4B-PH-K_1x04_P2.00mm_Horizontal"
+		(property "Footprint" "Connector_JST:JST_SH_SM04B-SRSS-TB_1x04-1MP_P1.00mm_Horizontal"
 			(at 153.67 118.11 0)
 			(effects
@@
 			(project "fimur-electrical-v0-2"
 				(path "/d9ca54f7-b1e2-4ace-986c-e50c0b614954"
-					(reference "J8")
+					(reference "J9")
 					(unit 1)
 				)
@@
 		(dnp no)
 		(fields_autoplaced yes)
-		(property "Reference" "J7"
+		(property "Reference" "J8"
 			(at 129.54 113.0299 0)
 			(effects
@@
 			)
 		)
-		(property "Footprint" "Connector_JST:JST_PH_S4B-PH-K_1x04_P2.00mm_Horizontal"
+		(property "Footprint" "Connector_JST:JST_SH_SM04B-SRSS-TB_1x04-1MP_P1.00mm_Horizontal"
 			(at 127 113.03 0)
 			(effects
@@
 			(project "fimur-electrical-v0-2"
 				(path "/d9ca54f7-b1e2-4ace-986c-e50c0b614954"
-					(reference "J7")
+					(reference "J8")
 					(unit 1)
 				)
@@
 		(dnp no)
 		(fields_autoplaced yes)
-		(property "Reference" "J11"
+		(property "Reference" "J12"
 			(at 156.21 139.6999 0)
 			(effects
@@
 			)
 		)
-		(property "Footprint" "Connector_JST:JST_PH_S4B-PH-K_1x04_P2.00mm_Horizontal"
+		(property "Footprint" "Connector_JST:JST_SH_SM04B-SRSS-TB_1x04-1MP_P1.00mm_Horizontal"
 			(at 153.67 139.7 0)
 			(effects
@@
 			(project "fimur-electrical-v0-2"
 				(path "/d9ca54f7-b1e2-4ace-986c-e50c0b614954"
-					(reference "J11")
+					(reference "J12")
 					(unit 1)
 				)
@@
 		(dnp no)
 		(fields_autoplaced yes)
-		(property "Reference" "J12"
+		(property "Reference" "J13"
 			(at 182.88 144.7799 0)
 			(effects
@@
 			)
 		)
-		(property "Footprint" "Connector_JST:JST_PH_S4B-PH-K_1x04_P2.00mm_Horizontal"
+		(property "Footprint" "Connector_JST:JST_SH_SM04B-SRSS-TB_1x04-1MP_P1.00mm_Horizontal"
 			(at 180.34 144.78 0)
 			(effects
@@
 			(project "fimur-electrical-v0-2"
 				(path "/d9ca54f7-b1e2-4ace-986c-e50c0b614954"
-					(reference "J12")
+					(reference "J13")
+					(unit 1)
+				)
+			)
+		)
+	)
+	(symbol
+		(lib_id "power:VCC")
+		(at 35.56 87.63 180)
+		(unit 1)
+		(exclude_from_sim no)
+		(in_bom yes)
+		(on_board yes)
+		(dnp no)
+		(property "Reference" "#PWR02"
+			(at 35.56 83.82 0)
+			(effects
+				(font
+					(size 1.27 1.27)
+				)
+				(hide yes)
+			)
+		)
+		(property "Value" "VCC"
+			(at 33.782 86.36 0)
+			(effects
+				(font
+					(size 1.27 1.27)
+				)
+			)
+		)
+		(property "Footprint" ""
+			(at 35.56 87.63 0)
+			(effects
+				(font
+					(size 1.27 1.27)
+				)
+				(hide yes)
+			)
+		)
+		(property "Datasheet" ""
+			(at 35.56 87.63 0)
+			(effects
+				(font
+					(size 1.27 1.27)
+				)
+				(hide yes)
+			)
+		)
+		(property "Description" "Power symbol creates a global label with name \"VCC\""
+			(at 35.56 87.63 0)
+			(effects
+				(font
+					(size 1.27 1.27)
+				)
+				(hide yes)
+			)
+		)
+		(pin "1"
+		)
+		(instances
+			(project ""
+				(path "/d9ca54f7-b1e2-4ace-986c-e50c0b614954"
+					(reference "#PWR02")
 					(unit 1)
 				)
@@
 		(dnp no)
 		(fields_autoplaced yes)
-		(property "Reference" "J15"
+		(property "Reference" "J7"
 			(at 105.41 101.5999 0)
 			(effects
@@
 			)
 		)
-		(property "Footprint" "Connector_JST:JST_PH_S4B-PH-K_1x04_P2.00mm_Horizontal"
+		(property "Footprint" "Connector_JST:JST_SH_SM04B-SRSS-TB_1x04-1MP_P1.00mm_Horizontal"
 			(at 102.87 101.6 0)
 			(effects
@@
 			(project "fimur-electrical-v0-2"
 				(path "/d9ca54f7-b1e2-4ace-986c-e50c0b614954"
-					(reference "J15")
+					(reference "J7")
 					(unit 1)
 				)
@@
 	(symbol
 		(lib_id "power:GND")
-		(at 36.83 160.02 0)
+		(at 36.83 85.09 180)
 		(unit 1)
 		(exclude_from_sim no)
@@
 		(on_board yes)
 		(dnp no)
-		(fields_autoplaced yes)
 		(property "Reference" "#PWR01"
-			(at 36.83 166.37 0)
+			(at 36.83 78.74 0)
 			(effects
 				(font
@@
 		)
 		(property "Value" "GND"
-			(at 36.83 165.1 0)
+			(at 34.798 81.534 0)
 			(effects
 				(font
 					(size 1.27 1.27)
 				)
+				(justify right)
 			)
 		)
 		(property "Footprint" ""
-			(at 36.83 160.02 0)
+			(at 36.83 85.09 0)
 			(effects
 				(font
@@
 		)
 		(property "Datasheet" ""
-			(at 36.83 160.02 0)
+			(at 36.83 85.09 0)
 			(effects
 				(font
@@
 		)
 		(property "Description" "Power symbol creates a global label with name \"GND\" , ground"
-			(at 36.83 160.02 0)
+			(at 36.83 85.09 0)
 			(effects
 				(font
@@
 		)
 		(instances
-			(project ""
+			(project "fimur-electrical-v0-2"
 				(path "/d9ca54f7-b1e2-4ace-986c-e50c0b614954"
 					(reference "#PWR01")
@@
 			)
 		)
-		(property "Footprint" "Connector_PinSocket_1.27mm:PinSocket_2x02_P1.27mm_Vertical"
+		(property "Footprint" "Connector_PinSocket_2.54mm:PinSocket_2x02_P2.54mm_Vertical"
 			(at 41.91 107.95 0)
 			(effects
@@
 		(dnp no)
 		(fields_autoplaced yes)
-		(property "Reference" "J10"
+		(property "Reference" "J11"
 			(at 209.55 128.2699 0)
 			(effects
@@
 			)
 		)
-		(property "Footprint" "Connector_JST:JST_PH_S4B-PH-K_1x04_P2.00mm_Horizontal"
+		(property "Footprint" "Connector_JST:JST_SH_SM04B-SRSS-TB_1x04-1MP_P1.00mm_Horizontal"
 			(at 207.01 128.27 0)
 			(effects
@@
 			(project "fimur-electrical-v0-2"
 				(path "/d9ca54f7-b1e2-4ace-986c-e50c0b614954"
-					(reference "J10")
+					(reference "J11")
 					(unit 1)
 				)
@@
 			)
 		)
-		(property "Footprint" "Connector_JST:JST_PH_S4B-PH-K_1x04_P2.00mm_Horizontal"
+		(property "Footprint" "Connector_JST:JST_SH_SM04B-SRSS-TB_1x04-1MP_P1.00mm_Horizontal"
 			(at 78.74 95.25 0)
 			(effects
@@
 		(dnp no)
 		(fields_autoplaced yes)
-		(property "Reference" "J9"
+		(property "Reference" "J10"
 			(at 182.88 123.1899 0)
 			(effects
@@
 			)
 		)
-		(property "Footprint" "Connector_JST:JST_PH_S4B-PH-K_1x04_P2.00mm_Horizontal"
+		(property "Footprint" "Connector_JST:JST_SH_SM04B-SRSS-TB_1x04-1MP_P1.00mm_Horizontal"
 			(at 180.34 123.19 0)
 			(effects
@@
 			(project "fimur-electrical-v0-2"
 				(path "/d9ca54f7-b1e2-4ace-986c-e50c0b614954"
-					(reference "J9")
+					(reference "J10")
 					(unit 1)
 				)
