File: electrical/fimur-electrical-v0-2/fimur-electrical-v0-2.kicad_pcb (KiCad board)
At the start: 2 copper layers, 73 x 47.5 mm, 30 parts, among them J1 Conn_01x16, J10 Conn_01x04, J11 Conn_01x04, J12 Conn_01x04, J13 Conn_01x04, J14 Conn_01x04, J15 Conn_01x04, J17 Conn_02x02_Odd_Even, J2 Conn_01x16, J3 Conn_01x03_Pin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

Commit message: all kicad files for v0 boards
Parts:
- removed J17: Conn_02x02_Odd_Even, Connector_PinSocket_2.54mm:PinSocket_2x02_P2.54mm_Vertical
- added GND: TestPoint_Loop_D1.80mm_Drill1.0mm_Beaded, TestPoint:TestPoint_Loop_D1.80mm_Drill1.0mm_Beaded, F.Cu at (152.5, 119.0)
- added J16: HC-PZ254-11.5L-1x2PZ, Connector_PinHeader_2.54mm:PinHeader_1x02_P2.54mm_Vertical, F.Cu at (155.8, 115.0)
- added REF**: MountingHole_2.2mm_M2, MountingHole:MountingHole_2.2mm_M2, F.Cu at (126.8, 117.8)
- added REF**: MountingHole_2.2mm_M2, MountingHole:MountingHole_2.2mm_M2, F.Cu at (147.2, 117.8)
- added REF**: MountingHole_2.2mm_M2, MountingHole:MountingHole_2.2mm_M2, F.Cu at (126.8, 105.2)
- added REF**: MountingHole_2.2mm_M2, MountingHole:MountingHole_2.2mm_M2, F.Cu at (147.2, 105.2)
- added VCC: TestPoint_Loop_D1.80mm_Drill1.0mm_Beaded, TestPoint:TestPoint_Loop_D1.80mm_Drill1.0mm_Beaded, F.Cu at (152.5, 127.5)
- J1, J2: value Conn_01x16 -> 2541FV-16P-B
- J10, J11, J12, J13, J14, J15, J6, J7, J8, J9: value Conn_01x04 -> XY-SM04B-SRSS-TB
- J3, J4, J5: value Conn_01x03_Pin -> PZ254V-11-03P-A40; footprint Connector_PinSocket_2.54mm:PinSocket_1x03_P2.54mm_Vertical -> Connector_PinHeader_2.54mm:PinHeader_1x03_P2.54mm_Vertical
- moved J1 29.8 mm to (119.1, 100.0), turned to 0 degrees
- moved J2 29.8 mm to (119.1, 122.9), turned to 0 degrees
- moved R2 7.57 mm to (140.0, 118.0), turned to -90 degrees
- moved R1 5.26 mm to (142.5, 118.0), turned to -90 degrees
- moved J3 2.54 mm to (154.5, 109.6), turned to 0 degrees
- moved J4 2.54 mm to (154.5, 105.0), turned to 0 degrees
- moved J5 2.54 mm to (154.5, 100.4), turned to 0 degrees
- moved REF** 0.20 mm to (137.0, 111.5)
- turned U1 to 180 degrees
Connections:
- R1 pad 1: VCC -> Net-(J16-Pin_2)
- R1 pad 2: Net-(J17-Pin_2) -> Net-(J1-2)
- R2 pad 1: VCC -> Net-(J16-Pin_2)
- R2 pad 2: Net-(J17-Pin_4) -> Net-(J1-3)
Routing:
- net Net-(J16-Pin_2): track 0.00 -> 19.4 mm
- net VCC: track 324.3 -> 313.2 mm
- net Net-(J1-2): track 94.4 -> 83.7 mm
- net Net-(J1-3): track 93.4 -> 84.1 mm
- net Net-(J17-Pin_4): track 4.95 -> 0.00 mm
- net Net-(J17-Pin_2): track 4.93 -> 0.00 mm
- net GND: track 16.7 -> 12.6 mm
- net Net-(J12-Pin_3): track 31.5 -> 34.7 mm
- net Net-(J12-Pin_4): track 31.8 -> 34.5 mm
Other:
- board text added: "1.27cm"
- board text added: "2.032cm"
- board text added: "2cm"
- board text added: "4cm"
- board text added: "ADDR 0"
- board text added: "ADDR 1"
- board text added: "ADDR 2"
- board text added: "CH0"
- board text added: "CH1"
- board text added: "CH2"
- board text added: "CH3"
- board text added: "CH4"
- board text added: "CH5"
- board text added: "CH6"
- board text added: "CH7"
- board text added: "GVDC"
- board text added: "MAINx2"
- board text added: "PULLUP"
- board text added: "fimur 0.2.1 i2c multiplex VCC: 3.3V"
