File: electrical/fimur-electrical-v0-2/fimur-electrical-v0-2.kicad_sch (KiCad schematic)
At the start: 20 parts, among them J1 Conn_01x16, J10 Conn_01x04, J11 Conn_01x04, J12 Conn_01x04, J13 Conn_01x04, J14 Conn_01x04, J15 Conn_01x04, J17 Conn_02x02_Odd_Even, J2 Conn_01x16, J3 Conn_01x03_Pin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

Commit message: all kicad files for v0 boards
Parts:
- removed J17: Conn_02x02_Odd_Even, Connector_PinSocket_2.54mm:PinSocket_2x02_P2.54mm_Vertical, symbol Connector_Generic:Conn_02x02_Odd_Even
- added J16: HC-PZ254-11.5L-1x2PZ, Connector_PinHeader_2.54mm:PinHeader_1x02_P2.54mm_Vertical, symbol Connector_Generic:Conn_01x02
- J1, J2: value Conn_01x16 -> 2541FV-16P-B
- J10, J11, J12, J13, J14, J15, J6, J7, J8, J9: value Conn_01x04 -> XY-SM04B-SRSS-TB
- J3, J4, J5: value Conn_01x03_Pin -> PZ254V-11-03P-A40; footprint Connector_PinSocket_2.54mm:PinSocket_1x03_P2.54mm_Vertical -> Connector_PinHeader_2.54mm:PinHeader_1x03_P2.54mm_Vertical
Connections:
- net VCC: now also J16.1 (Pin_1); no longer R1.1, R2.1
- net at J1.12 (2), J6.3 (Pin_3), J7.3 (Pin_3)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: now also R1.2
- net at J1.13 (3), J6.4 (Pin_4), J7.4 (Pin_4)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: now also R2.2
- new net: J16.2 (Pin_2), R1.1, R2.1
Other:
- moved on the sheet: R1, R2, R3
