File: electrical/fimur-electrical-v0-2/fimur-electrical-v0-1/fimur-electrical-v0-1.kicad_pcb (KiCad board)
At the start: 2 copper layers, 47 x 27 mm, 21 parts, among them J1 Conn_01x04_Pin, J2 Conn_01x04_Pin, J3 Conn_02x02_Odd_Even, U1 NCP163AFCS180T2G, U2 ICM-20948, U3 ICM-20948

Commit message: all kicad files for v0 boards
Parts:
- removed J3: Conn_02x02_Odd_Even, Connector_PinSocket_2.54mm:PinSocket_2x02_P2.54mm_Horizontal
- added J4: Conn_01x02, Connector_PinHeader_2.54mm:PinHeader_1x02_P2.54mm_Horizontal, F.Cu at (95.3, 93.5)
- added J5: Conn_01x02, Connector_PinHeader_2.54mm:PinHeader_1x02_P2.54mm_Horizontal, F.Cu at (102.2, 93.5)
- moved R1 3.54 mm to (104.0, 98.5)
- moved R2 3.54 mm to (106.5, 98.5)
Routing:
- net Net-(J5-Pin_1): track 32.7 -> 43.3 mm
- net Net-(J4-Pin_2): track 7.02 -> 12.1 mm
- net Net-(J1-Pin_4): track 46.8 -> 50.6 mm
- net Net-(J4-Pin_1): track 74.9 -> 71.1 mm
- net GND: track 25.8 -> 27.6 mm
- net Net-(J1-Pin_3): track 51.7 -> 52.8 mm
Other:
- board text added: "GVDC"
- board text added: "MAIN"
- board text added: "fimur 0.1.1 2x ICM20948 IMU VCC: 2.2 - 5.5V i2c"
- board text removed: "VCC: 2.2 - 5.5V"
- board text removed: "fimur 0.1.1"
