File: electrical/fimur-electrical-v0-2/fimur-electrical-v0-1/fimur-electrical-v0-1.kicad_sch (KiCad schematic)
At the start: 14 parts, among them J1 Conn_01x04_Pin, J2 Conn_01x04_Pin, J3 Conn_02x02_Odd_Even, U1 NCP163AFCS180T2G, U2 ICM-20948, U3 ICM-20948

Commit message: all kicad files for v0 boards
Parts:
- removed J3: Conn_02x02_Odd_Even, Connector_PinSocket_2.54mm:PinSocket_2x02_P2.54mm_Horizontal, symbol Connector_Generic:Conn_02x02_Odd_Even
- added J4, J5: Conn_01x02, Connector_PinHeader_2.54mm:PinHeader_1x02_P2.54mm_Horizontal, symbol Connector_Generic:Conn_01x02
Connections:
- net at C2.1, C3.1, C5.1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: now also J4.1 (Pin_1)
- net at R1.1, R2.1: now also J4.2 (Pin_2)
- net at U2.11 (FSYNC), U3.11 (FSYNC): now also J5.1 (Pin_1), J5.2 (Pin_2)
Changed lines of the file:
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@@
-	)
-	(junction
-		(at 83.82 87.63)
-		(diameter 0)
-		(color 0 0 0 0)
 	)
 	(junction
@@
 	)
 	(junction
-		(at 83.82 104.14)
-		(diameter 0)
-		(color 0 0 0 0)
-	)
-	(junction
 		(at 110.49 116.84)
-		(diameter 0)
-		(color 0 0 0 0)
-	)
-	(junction
-		(at 90.17 102.87)
 		(diameter 0)
 		(color 0 0 0 0)
@@
 	)
 	(junction
+		(at 77.47 104.14)
+		(diameter 0)
+		(color 0 0 0 0)
+	)
+	(junction
 		(at 228.6 69.85)
+		(diameter 0)
+		(color 0 0 0 0)
+	)
+	(junction
+		(at 92.71 99.06)
 		(diameter 0)
 		(color 0 0 0 0)
@@
 	)
 	(junction
+		(at 78.74 87.63)
+		(diameter 0)
+		(color 0 0 0 0)
+	)
+	(junction
 		(at 190.5 69.85)
 		(diameter 0)
@@
 	(wire
 		(pts
-			(xy 77.47 87.63) (xy 83.82 87.63)
+			(xy 77.47 87.63) (xy 78.74 87.63)
 		)
 		(stroke
@@
 	(wire
 		(pts
-			(xy 83.82 104.14) (xy 83.82 102.87)
-		)
-		(stroke
-			(width 0)
-			(type default)
-		)
-	)
-	(wire
-		(pts
 			(xy 49.53 118.11) (xy 83.82 118.11)
 		)
@@
 	(wire
 		(pts
-			(xy 90.17 102.87) (xy 91.44 102.87)
-		)
-		(stroke
-			(width 0)
-			(type default)
-		)
-	)
-	(wire
-		(pts
 			(xy 69.85 114.3) (xy 107.95 114.3)
 		)
@@
 	(wire
 		(pts
-			(xy 90.17 121.92) (xy 115.57 121.92)
+			(xy 92.71 121.92) (xy 115.57 121.92)
 		)
 		(stroke
@@
 	(wire
 		(pts
-			(xy 83.82 87.63) (xy 102.87 87.63)
+			(xy 78.74 87.63) (xy 102.87 87.63)
 		)
 		(stroke
@@
 	(wire
 		(pts
+			(xy 78.74 87.63) (xy 78.74 96.52)
+		)
+		(stroke
+			(width 0)
+			(type default)
+		)
+	)
+	(wire
+		(pts
 			(xy 30.48 87.63) (xy 30.48 102.87)
 		)
@@
 	(wire
 		(pts
+			(xy 92.71 99.06) (xy 93.98 99.06)
+		)
+		(stroke
+			(width 0)
+			(type default)
+		)
+	)
+	(wire
+		(pts
 			(xy 190.5 69.85) (xy 190.5 90.17)
 		)
@@
 	(wire
 		(pts
-			(xy 90.17 90.17) (xy 90.17 102.87)
-		)
-		(stroke
-			(width 0)
-			(type default)
-		)
-	)
-	(wire
-		(pts
-			(xy 90.17 102.87) (xy 90.17 121.92)
-		)
-		(stroke
-			(width 0)
-			(type default)
-		)
-	)
-	(wire
-		(pts
 			(xy 69.85 114.3) (xy 52.07 114.3)
 		)
@@
 	(wire
 		(pts
+			(xy 92.71 99.06) (xy 92.71 121.92)
+		)
+		(stroke
+			(width 0)
+			(type default)
+		)
+	)
+	(wire
+		(pts
 			(xy 220.98 105.41) (xy 220.98 114.3)
 		)
@@
 	(wire
 		(pts
-			(xy 83.82 87.63) (xy 83.82 90.17)
-		)
-		(stroke
-			(width 0)
-			(type default)
-		)
-	)
-	(wire
-		(pts
 			(xy 228.6 69.85) (xy 228.6 97.79)
 		)
@@
 	(wire
 		(pts
+			(xy 92.71 96.52) (xy 92.71 99.06)
+		)
+		(stroke
+			(width 0)
+			(type default)
+		)
+	)
+	(wire
+		(pts
 			(xy 30.48 102.87) (xy 25.4 102.87)
 		)
@@
 	(wire
 		(pts
+			(xy 77.47 99.06) (xy 77.47 104.14)
+		)
+		(stroke
+			(width 0)
+			(type default)
+		)
+	)
+	(wire
+		(pts
 			(xy 33.02 92.71) (xy 50.8 92.71)
 		)
@@
 	(wire
 		(pts
+			(xy 78.74 99.06) (xy 77.47 99.06)
+		)
+		(stroke
+			(width 0)
+			(type default)
+		)
+	)
+	(wire
+		(pts
 			(xy 147.32 105.41) (xy 147.32 114.3)
 		)
@@
 	(wire
 		(pts
+			(xy 93.98 96.52) (xy 92.71 96.52)
+		)
+		(stroke
+			(width 0)
+			(type default)
+		)
+	)
+	(wire
+		(pts
 			(xy 111.76 87.63) (xy 111.76 118.11)
 		)
@@
 	(wire
 		(pts
-			(xy 90.17 90.17) (xy 86.36 90.17)
-		)
-		(stroke
-			(width 0)
-			(type default)
-		)
-	)
-	(wire
-		(pts
 			(xy 33.02 92.71) (xy 33.02 107.95)
 		)
@@
 	(wire
 		(pts
+			(xy 83.82 104.14) (xy 83.82 105.41)
+		)
+		(stroke
+			(width 0)
+			(type default)
+		)
+	)
+	(wire
+		(pts
 			(xy 134.62 69.85) (xy 154.94 69.85)
 		)
@@
 	(wire
 		(pts
-			(xy 86.36 102.87) (xy 90.17 102.87)
-		)
-		(stroke
-			(width 0)
-			(type default)
-		)
-	)
-	(wire
-		(pts
 			(xy 186.69 87.63) (xy 186.69 118.11)
 		)
@@
 		(pts
 			(xy 185.42 85.09) (xy 193.04 85.09)
-		)
-		(stroke
-			(width 0)
-			(type default)
-		)
-	)
-	(wire
-		(pts
-			(xy 83.82 104.14) (xy 83.82 105.41)
 		)
 		(stroke
@@
 	)
 	(symbol
-		(lib_id "Connector_Generic:Conn_02x02_Odd_Even")
-		(at 83.82 97.79 90)
+		(lib_id "Connector_Generic:Conn_01x02")
+		(at 83.82 96.52 0)
 		(unit 1)
 		(exclude_from_sim no)
@@
 		(on_board yes)
 		(dnp no)
-		(fields_autoplaced yes)
-		(property "Reference" "J3"
-			(at 88.9 95.2499 90)
-			(effects
-				(font
-					(size 1.27 1.27)
-				)
-				(justify right)
-			)
-		)
-		(property "Value" "Conn_02x02_Odd_Even"
-			(at 88.9 97.7899 90)
-			(effects
-				(font
-					(size 1.27 1.27)
-				)
-				(justify right)
-			)
-		)
-		(property "Footprint" "Connector_PinSocket_2.54mm:PinSocket_2x02_P2.54mm_Horizontal"
-			(at 83.82 97.79 0)
+		(property "Reference" "J4"
+			(at 79.756 91.186 0)
+			(effects
+				(font
+					(size 1.27 1.27)
+				)
+				(justify left)
+			)
+		)
+		(property "Value" "Conn_01x02"
+			(at 79.756 93.726 0)
+			(effects
+				(font
+					(size 1.27 1.27)
+				)
+				(justify left)
+			)
+		)
+		(property "Footprint" "Connector_PinHeader_2.54mm:PinHeader_1x02_P2.54mm_Horizontal"
+			(at 83.82 96.52 0)
 			(effects
 				(font
@@
 		)
 		(property "Datasheet" "~"
-			(at 83.82 97.79 0)
-			(effects
-				(font
-					(size 1.27 1.27)
-				)
-				(hide yes)
-			)
-		)
-		(property "Description" "Generic connector, double row, 02x02, odd/even pin numbering scheme (row 1 odd numbers, row 2 even numbers), script generated (kicad-library-utils/schlib/autogen/connector/)"
-			(at 83.82 97.79 0)
-			(effects
-				(font
-					(size 1.27 1.27)
-				)
-				(hide yes)
-			)
+			(at 83.82 96.52 0)
+			(effects
+				(font
+					(size 1.27 1.27)
+				)
+				(hide yes)
+			)
+		)
+		(property "Description" "Generic connector, single row, 01x02, script generated (kicad-library-utils/schlib/autogen/connector/)"
+			(at 83.82 96.52 0)
+			(effects
+				(font
+					(size 1.27 1.27)
+				)
+				(hide yes)
+			)
+		)
+		(pin "2"
 		)
 		(pin "1"
-		)
-		(pin "3"
-		)
-		(pin "2"
-		)
-		(pin "4"
 		)
 		(instances
 			(project ""
 				(path "/d9ca54f7-b1e2-4ace-986c-e50c0b614954"
-					(reference "J3")
+					(reference "J4")
 					(unit 1)
 				)
@@
 					(unit 1)
 				)
+			)
+		)
+	)
+	(symbol
+		(lib_id "Connector_Generic:Conn_01x02")
+		(at 99.06 96.52 0)
+		(unit 1)
+		(exclude_from_sim no)
+		(in_bom yes)
+		(on_board yes)
+		(dnp no)
+		(property "Reference" "J5"
+			(at 94.996 91.44 0)
+			(effects
+				(font
+					(size 1.27 1.27)
+				)
+				(justify left)
+			)
+		)
+		(property "Value" "Conn_01x02"
+			(at 94.996 93.98 0)
+			(effects
+				(font
+					(size 1.27 1.27)
+				)
+				(justify left)
+			)
+		)
+		(property "Footprint" "Connector_PinHeader_2.54mm:PinHeader_1x02_P2.54mm_Horizontal"
+			(at 99.06 96.52 0)
+			(effects
+				(font
+					(size 1.27 1.27)
+				)
+				(hide yes)
+			)
+		)
+		(property "Datasheet" "~"
+			(at 99.06 96.52 0)
+			(effects
+				(font
+					(size 1.27 1.27)
+				)
+				(hide yes)
+			)
+		)
+		(property "Description" "Generic connector, single row, 01x02, script generated (kicad-library-utils/schlib/autogen/connector/)"
+			(at 99.06 96.52 0)
+			(effects
+				(font
+					(size 1.27 1.27)
+				)
+				(hide yes)
+			)
+		)
+		(pin "2"
+		)
+		(pin "1"
+		)
+		(instances
+			(project "fimur-electrical-v0-1"
+				(path "/d9ca54f7-b1e2-4ace-986c-e50c0b614954"
+					(reference "J5")
+					(unit 1)
+				)
