File: electrical/v0/v0-2/fimur-electrical-v0-2.kicad_pcb (KiCad board)
At the start: 2 copper layers, 73 x 47.5 mm, 36 parts, among them J1 2541FV-16P-B, J10 XY-SM04B-SRSS-TB, J11 XY-SM04B-SRSS-TB, J12 XY-SM04B-SRSS-TB, J13 XY-SM04B-SRSS-TB, J14 XY-SM04B-SRSS-TB, J15 XY-SM04B-SRSS-TB, J16 HC-PZ254-11.5L-1x2PZ, J2 2541FV-16P-B, J3 PZ254V-11-03P-A40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

Commit message: v2 of multiplex board
Parts:
- J3, J4, J5: value PZ254V-11-03P-A40 -> HC-PZ254-11.5L-1x3PZ
- moved J8 1.70 mm to (91.5, 126.2)
- moved J15 1.20 mm to (91.4, 96.8)
- moved REF** 0.20 mm to (137.0, 111.3)
- turned U1 to 0 degrees
Routing:
- net VCC: track 313.2 -> 316.9 mm
- net GND: track 12.6 -> 14.2 mm
- net Net-(J15-Pin_3): track 30.6 -> 31.9 mm
- net Net-(J15-Pin_4): track 29.6 -> 30.5 mm
- net Net-(U1-~{RESET}): track 5.65 -> 4.91 mm
Other:
- board text added: "DN"
- board text added: "UP"
- board text added: "fimur 0.2.2 i2c multiplex VCC: 3.3V"
- board text removed: "fimur 0.2.1 i2c multiplex VCC: 3.3V"
