File: electrical/v0/v0-2/fimur-electrical-v0-2.kicad_sch (KiCad schematic)
At the start: 20 parts, among them J1 2541FV-16P-B, J10 XY-SM04B-SRSS-TB, J11 XY-SM04B-SRSS-TB, J12 XY-SM04B-SRSS-TB, J13 XY-SM04B-SRSS-TB, J14 XY-SM04B-SRSS-TB, J15 XY-SM04B-SRSS-TB, J16 HC-PZ254-11.5L-1x2PZ, J2 2541FV-16P-B, J3 PZ254V-11-03P-A40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

Commit message: v2 of multiplex board
Parts:
- J3, J4, J5: value PZ254V-11-03P-A40 -> HC-PZ254-11.5L-1x3PZ
Changed lines of the file:
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@@
 			)
 		)
-		(property "Value" "PZ254V-11-03P-A40"
+		(property "Value" "HC-PZ254-11.5L-1x3PZ"
 			(at 45.085 147.32 0)
 			(effects
@@
 			)
 		)
-		(property "Value" "PZ254V-11-03P-A40"
+		(property "Value" "HC-PZ254-11.5L-1x3PZ"
 			(at 75.565 147.32 0)
 			(effects
@@
 			)
 		)
-		(property "Value" "PZ254V-11-03P-A40"
+		(property "Value" "HC-PZ254-11.5L-1x3PZ"
 			(at 60.325 147.32 0)
 			(effects
